File: hw/kicad/minix-box.kicad_pcb (KiCad board)
At the start: 2 copper layers, 0 parts

Commit message: Add placeholder board outline to pass DRC
Empty PCB without Edge.Cuts edges triggers a DRC violation in
KiCad 10. Add a 50x20mm placeholder rectangle that will be replaced
with the actual board outline during layout.

Co-Authored-By: Claude Opus 4.6 <noreply@anthropic.com>
Other:
- board outline added: 50 x 20 mm
Changed lines of the file:
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@@
 	)
 	(net 0 "")
+	(gr_rect
+		(start 100 100)
+		(end 150 120)
+		(stroke (width 0.05) (type default))
+		(fill none)
+		(layer "Edge.Cuts")
+	)
 )
