File: hw/kicad/minix-box.kicad_sch (KiCad schematic)
At the start: 0 parts

Commit message: Add components to schema
Parts:
- added Card1: TF-01A, easyeda2kicad:TF-SMD_TF-01A, symbol easyeda2kicad:TF-01A
- added D1, D2: LED, symbol Device:LED
- added J1, J2: USB_C_Receptacle_USB2.0_16P, symbol Connector:USB_C_Receptacle_USB2.0_16P
- added SW1, SW2: SW_Push, symbol Switch:SW_Push
- added U1: F1C200S, easyeda2kicad:QFN-88_L10.0-W10.0-P0.40-BL-EP6.75, symbol easyeda2kicad:F1C200S
- added U2: CH340N, Package_SO:JEITA_SOIC-8_3.9x4.9mm_P1.27mm, symbol Interface_USB:CH340N
- added U3: W25Q128JVSIQTR, easyeda2kicad:SOIC-8_L5.3-W5.3-P1.27-LS8.0-BL, symbol easyeda2kicad:W25Q128JVSIQTR
- added U4, U5: SY8089AAAC, easyeda2kicad:SOT-23-5_L3.0-W1.7-P0.95-LS2.8-BR, symbol easyeda2kicad:SY8089AAAC
- added Y1, Y2: Crystal, symbol Device:Crystal
Connections:
- new net: J1.A1 (GND), J1.A12 (GND), J1.B1 (GND), J1.B12 (GND)
- new net: J1.A4 (VBUS), J1.A9 (VBUS), J1.B4 (VBUS), J1.B9 (VBUS)
- new net: J2.A1 (GND), J2.A12 (GND), J2.B1 (GND), J2.B12 (GND)
- new net: J2.A4 (VBUS), J2.A9 (VBUS), J2.B4 (VBUS), J2.B9 (VBUS)
